Commit message: added gazebo
added diff_drive and lidar

File: urdf/my_robot.xacro (robot description, xacro)
@@ -1,123 +1,256 @@
 <?xml version="1.0" encoding="UTF-8"?>
-<robot name ="multipleshapes">
+<!-- <robot name="myRobot"> -->
+<robot xmlns:xacro="http://www.ros.org/wiki/xacro" name="myRobot">
+    <!-- <xacro:include filename="inertial_macros.xacro"/> -->
     <material name="blue">
-        <color rgba="0 0 1 1"/>
+        <color rgba="0 0 1 1" />
     </material>
     <material name="white">
-        <color rgba="1 1 1 1"/>
+        <color rgba="1 1 1 1" />
     </material>
-    <link name= "base_link">
-        <visual>
-            <geometry>
-                <box size="0.9 1.6 0.4"/>
-            </geometry>
-            <origin rpy="0.0 0.0 0.0" xyz="0.0 0.0 0.3"/>
+    <material name="black">
+        <color rgba="0 0 0 0" />
+    </material>
+    <link name="base_footprint"></link>
+    <joint name="base_to_footprint_joint" type="fixed">
+        <origin xyz="0.0 0.0 0.15" rpy="0.0 0.0 0.0" />
+        <parent link="base_footprint" />
+        <child link="base_link" />
+    </joint>
+    <!-- BASE LINK -->
+    <link name="base_link">
+        <visual>
+            <geometry>
+                <cylinder radius="0.5" length="1.3" />
+            </geometry>
+            <origin rpy="0.0 0.0 0.0" xyz="0.0 0.0 0.9" />
             <material name="blue">
             </material>
         </visual>
-    </link>
-    <link name="front_left">
-        <visual>
-            <geometry>
-                <sphere radius="0.1"/>
-            </geometry>
-            <origin xyz="-0.24 0.7 -0.5" rpy="0.0 0.0 0.0"/>
-        </visual>
-    </link>
-    <joint name="base_to_frontleft" type="fixed">
-        <origin xyz="0.0 0.0 0.0" rpy="1.0 0.0 0.0"/>
-        <parent link="base_link"/>
-        <child link="front_left"/>
-    </joint>
-    <link name="front_right">
-        <visual>
-            <geometry>
-                <sphere radius="0.1"/>
-            </geometry>
-            <origin xyz="0.24 0.7 -0.5" rpy="0.0 0.0 0.0"/>
-        </visual>
-    </link>
-    <joint name="base_to_frontright" type="fixed">
-        <origin xyz="0.0 0.0 0.0" rpy="1.0 0.0 0.0"/>
-        <parent link="base_link"/>
-        <child link="front_right"/>
-    </joint>
-    <link name="front_link">
-        <visual>
-            <geometry>
-                <box size="0.1 0.1 1.3"/>
-            </geometry>
-            <origin xyz="-0.1 0.0 0.0" rpy="0.0 0.0 0.0"/>
-        </visual>
-    </link>
-    <joint name="base_to_front" type="fixed">
-        <origin xyz="0.0 0.5 0.0" rpy="0.0 1.57075 0.0"/>
-        <parent link="base_link"/>
-        <child link="front_link"/>
-    </joint>
-    <link name="back_link">
-        <visual>
-            <geometry>
-                <box size="0.1 0.1 1.3"/>
-            </geometry>
-            <origin xyz="-0.1 0.0 0.0" rpy="0.0 0.0 0.0"/>
-        </visual>
-    </link>
-    <joint name="base_to_back" type="fixed">
-        <origin xyz="0.0 -0.5 0.0" rpy="0.0 1.57075 0.0"/>
-        <parent link="base_link"/>
-        <child link="back_link"/>
-    </joint>
-    <link name = "front_right_wheel">
-        <visual>
-            <geometry>
-                <cylinder radius="0.17" length="0.15"/>
-            </geometry>
-            <origin rpy="0.0 0.0 0.0" xyz="-0.13 0.0 0.6"/>
+        <collision>
+            <geometry>
+                <cylinder radius="0.5" length="1.3" />
+            </geometry>
+            <origin rpy="0.0 0.0 0.0" xyz="0.0 0.0 0.9" />
+        </collision>
+        <inertial>
+            <mass value="10.0" />
+            <inertia ixx="1.0" ixy="0.0" ixz="0.0" iyy="1.0" iyz="0.0" izz="1.0" />
+        </inertial>
+    </link>
+    <!-- HEAD LİNK -->
+    <link name="head_link">
+        <visual>
+            <geometry>
+                <sphere radius="0.5" />
+            </geometry>
+            <material name="white">
+            </material>
+        </visual>
+        <collision>
+            <geometry>
+                <sphere radius="0.5" />
+            </geometry>
+        </collision>
+        <inertial>
+            <mass value="2.0" />
+            <inertia ixx="1.0" ixy="0.0" ixz="0.0" iyy="1.0" iyz="0.0" izz="1.0" />
+        </inertial>
+    </link>
+    <joint name="base_to_head_joint" type="fixed">
+        <origin xyz="0.0 0.0 1.5" rpy="0.0 0.0 0.0" />
+        <parent link="base_link" />
+        <child link="head_link" />
+    </joint>
+    <!-- HEAD EYES -->
+    <link name="head_left_link">
+        <visual>
+            <geometry>
+                <sphere radius="0.1" />
+            </geometry>
+        </visual>
+        <collision>
+            <geometry>
+                <sphere radius="0.1" />
+            </geometry>
+        </collision>
+        <inertial>
+            <mass value="0.5" />
+            <inertia ixx="1.0" ixy="0.0" ixz="0.0" iyy="1.0" iyz="0.0" izz="1.0" />
+        </inertial>
+    </link>
+    <joint name="base_to_head_left_joint" type="fixed">
+        <origin xyz="-0.17 0.5 1.7" rpy="0.0 0.0 0.0" />
+        <parent link="base_link" />
+        <child link="head_left_link" />
+    </joint>
+    <link name="head_right_link">
+        <visual>
+            <geometry>
+                <sphere radius="0.1" />
+            </geometry>
+        </visual>
+        <collision>
+            <geometry>
+                <sphere radius="0.1" />
+            </geometry>
+        </collision>
+        <inertial>
+            <mass value="0.5" />
+            <inertia ixx="1.0" ixy="0.0" ixz="0.0" iyy="1.0" iyz="0.0" izz="1.0" />
+        </inertial>
+    </link>
+    <joint name="base_to_head_right_joint" type="fixed">
+        <origin xyz="0.17 0.5 1.7" rpy="0.0 0.0 0.0" />
+        <parent link="base_link" />
+        <child link="head_right_link" />
+    </joint>
+    <!-- BACK LEG LINK -->
+    <link name="back_leg_link">
+        <visual>
+            <geometry>
+                <box size="0.1 0.1 0.2" />
+            </geometry>
+        </visual>
+        <collision>
+            <geometry>
+                <box size="0.1 0.1 0.2" />
+            </geometry>
+        </collision>
+        <inertial>
+            <mass value="2.0" />
+            <inertia ixx="1.0" ixy="0.0" ixz="0.0" iyy="1.0" iyz="0.0" izz="1.0" />
+        </inertial>
+    </link>
+    <joint name="base_to_back_leg_joint" type="fixed">
+        <origin xyz="0.0 -0.3 0.2" rpy="0.0 0.0 0.0" />
+        <parent link="base_link" />
+        <child link="back_leg_link" />
+    </joint>
+    <!-- BACK LEG BASE LINK -->
+    <link name="back_leg_base_link">
+        <visual>
+            <geometry>
+                <box size="0.5 0.1 0.1" />
+            </geometry>
+        </visual>
+        <collision>
+            <geometry>
+                <box size="0.5 0.1 0.1" />
+            </geometry>
+        </collision>
+        <inertial>
+            <mass value="2.0" />
+            <inertia ixx="1.0" ixy="0.0" ixz="0.0" iyy="1.0" iyz="0.0" izz="1.0" />
+        </inertial>
+    </link>
+    <joint name="back_leg_to_leg_base_joint" type="fixed">
+        <origin xyz="0.0 0.0 -0.08" rpy="0.0 0.0 0.0" />
+        <parent link="back_leg_link" />
+        <child link="back_leg_base_link" />
+    </joint>
+    <!-- RIGHT WHEEL LINK -->
+    <link name="right_wheel_link">
+        <visual>
+            <pose relative_to='__model__'>0.0 0 0.0 0 0 0</pose>
+            <geometry>
+                <cylinder radius="0.12" length="0.12" />
+            </geometry>
             <material name="white"></material>
         </visual>
-    </link>
-    <joint name="front_to_front_right_wheel" type="continuous">
-        <parent link="front_link"/>
-        <child link="front_right_wheel"/>
-    </joint>
-    <link name = "front_left_wheel">
-        <visual>
-            <geometry>
-                <cylinder radius="0.17" length="0.15"/>
-            </geometry>
-            <origin rpy="0.0 0.0 0.0" xyz="-0.13 0.0 -0.6"/>
+        <collision>
+            <geometry>
+                <cylinder radius="0.12" length="0.12" />
+            </geometry>
+        </collision>
+        <inertial>
+            <mass value="1.0" />
+            <inertia ixx="1.0" ixy="0.0" ixz="0.0" iyy="1.0" iyz="0.0" izz="1.0" />
+        </inertial>
+    </link>
+    <joint name="leg_base_to_right_wheel_joint" type="continuous">
+        <parent link="back_leg_base_link" />
+        <child link="right_wheel_link" />
+        <origin xyz="0.3 0.0 0.0" rpy="0.0 1.57075 0.0" />
+        <axis xyz="0.0 0.0 1.0" />
+    </joint>
+    <!-- LEFT WHEEL LINK -->
+    <link name="left_wheel_link">
+        <visual>
+            <geometry>
+                <cylinder radius="0.12" length="0.12" />
+            </geometry>
             <material name="white"></material>
         </visual>
-    </link>
-    <joint name="front_to_front_left_wheel" type="continuous">
-        <parent link="front_link"/>
-        <child link="front_left_wheel"/>
-    </joint>
-    <link name = "back_right_wheel">
-        <visual>
-            <geometry>
-                <cylinder radius="0.17" length="0.15"/>
-            </geometry>
-            <origin rpy="0.0 0.0 0.0" xyz="-0.13 0.0 0.6"/>
+        <collision>
+            <geometry>
+                <cylinder radius="0.12" length="0.12" />
+            </geometry>
+        </collision>
+        <inertial>
+            <mass value="1.0" />
+            <inertia ixx="1.0" ixy="0.0" ixz="0.0" iyy="1.0" iyz="0.0" izz="1.0" />
+        </inertial>
+    </link>
+    <joint name="leg_base_to_left_wheel_joint" type="continuous">
+        <parent link="back_leg_base_link" />
+        <child link="left_wheel_link" />
+        <origin xyz="-0.3 0.0 0.0" rpy="0.0 1.57075 0.0" />
+        <axis xyz="0.0 0.0 1.0" />
+        <!-- <limit effort="100.0" velocity="100.0"/>
+        <dynamics damping="0.0" friction="0.5"/> -->
+    </joint>
+    <!-- FRONT LEG LINK -->
+    <link name="front_leg_link">
+        <visual>
+            <geometry>
+                <box size="0.1 0.1 0.2" />
+            </geometry>
+        </visual>
+        <collision>
+            <geometry>
+                <box size="0.1 0.1 0.2" />
+            </geometry>
+        </collision>
+        <inertial>
+            <mass value="2.0" />
+            <inertia ixx="1.0" ixy="0.0" ixz="0.0" iyy="1.0" iyz="0.0" izz="1.0" />
+        </inertial>
+    </link>
+    <joint name="base_to_front_leg_joint" type="fixed">
+        <origin xyz="0.0 0.3 0.2" rpy="0.0 0.0 0.0" />
+        <parent link="base_link" />
+        <child link="front_leg_link" />
+    </joint>
+    <!-- CASTER WHEEL LINK -->
+    <link name="caster_wheel_link">
+        <inertial>
+            <mass value="2.0"/>
+            <inertia ixx="1.0" ixy="0.0" ixz="0.0" iyy="1.0" iyz="0.0" izz="1.0"/>
+        </inertial>
+        <visual name="">
+            <geometry>
+                <sphere radius="0.13"/>
+            </geometry>
             <material name="white"></material>
         </visual>
-    </link>
-    <joint name="back_to_back_right_wheel" type="continuous">
-        <parent link="back_link"/>
-        <child link="back_right_wheel"/>
-    </joint>
-    <link name = "back_left_wheel">
-        <visual>
-            <geometry>
-                <cylinder radius="0.17" length="0.15"/>
-            </geometry>
-            <origin rpy="0.0 0.0 0.0" xyz="-0.13 0.0 -0.6"/>
-            <material name="white"></material>
-        </visual>
-    </link>
-    <joint name="back_to_back_left_wheel" type="continuous">
-        <parent link="back_link"/>
-        <child link="back_left_wheel"/>
+        <collision>
+            <surface>
+                <friction>
+                    <ode>
+                        <mu>0.0</mu>
+                    </ode>
+                </friction>
+            </surface>
+            <geometry>
+                <sphere radius="0.13"/>
+            </geometry>
+        </collision>
+    </link>
+    <joint name="front_leg_to_caster_joint" type="fixed">
+        <origin xyz="0.0 0.0 -0.09" rpy="0.0 0.0 0.0"/>
+        <parent link="front_leg_link"/>
+        <child link="caster_wheel_link"/>
+        <dynamics damping="0.0" friction="0.0"/>
     </joint>
 </robot>

File: urdf/my_robot3.urdf (robot description, URDF)
Before this commit: robot myRobot, 11 links, 10 joints
Links:
- removed link basefootprint
- removed link caster_wheels_link
- added link base_footprint
- added link caster_wheel_link, mass 2.0; collision sphere radius=0.12; visual sphere radius=0.12
- added link lidar_link, mass 0.5; collision box size=0.3 0.3 0.3; visual box size=0.2 0.2 0.15
Joints:
- removed joint base_to_leg_joint
- removed joint leg_base_to_left_wheel_joint
- removed joint leg_base_to_right_wheel_joint
- removed joint leg_to_leg_base_joint
- added joint back_leg_to_leg_base_joint: type fixed, parent back_leg_link, child back_leg_base_link, origin xyz=0.0 0.0 -0.08 rpy=0.0 0.0 0.0
- added joint base_to_back_leg_joint: type fixed, parent base_link, child back_leg_link, origin xyz=0.0 0.3 0.2 rpy=0.0 0.0 0.0
- added joint base_to_left_wheel_joint: type continuous, parent base_link, child left_wheel_link, origin xyz=0.3 0.3 0.11 rpy=0.0 1.57075 0.0, axis 0.0 0.0 1.0
- added joint base_to_lidar_joint: type fixed, parent base_link, child lidar_link, origin xyz=0.0 -0.6 0.25 rpy=0.0 0.0 0.0
- added joint base_to_right_wheel_joint: type continuous, parent base_link, child right_wheel_link, origin xyz=-0.3 0.3 0.11 rpy=0.0 1.57075 0.0, axis 0.0 0.0 1.0
- joint base_to_footprint_joint: parent basefootprint -> base_footprint
- joint base_to_front_leg_joint: origin xyz=0.0 0.3 0.2 rpy=0.0 0.0 0.0 -> xyz=0.0 -0.3 0.2 rpy=0.0 0.0 0.0
- joint base_to_head_left_joint: origin xyz=-0.17 0.5 1.7 rpy=0.0 0.0 0.0 -> xyz=0.17 -0.5 1.7 rpy=0.0 0.0 0.0
- joint base_to_head_right_joint: origin xyz=0.17 0.5 1.7 rpy=0.0 0.0 0.0 -> xyz=-0.17 -0.5 1.7 rpy=0.0 0.0 0.0
- joint front_leg_to_caster_joint: child caster_wheels_link -> caster_wheel_link
