Commit message: added map server and amcl localization

File: urdf/deneme.urdf (robot description, URDF)
Before this commit: robot myRobot, 12 links, 11 joints
Joints:
- joint back_leg_to_leg_base_joint: origin xyz=0.0 0.0 -0.08 rpy=0.0 0.0 1.57075 -> xyz=0.0 0.0 -0.08 rpy=0.0 0.0 0.0
- joint base_to_back_leg_joint: origin xyz=-0.3 0.0 0.2 rpy=0.0 0.0 0.0 -> xyz=0.0 0.3 0.2 rpy=0.0 0.0 0.0
- joint base_to_footprint_joint: origin xyz=0.0 0.0 0.0 rpy=0.0 0.0 0.0 -> xyz=0.0 0.0 0.15 rpy=0.0 0.0 0.0
- joint base_to_front_leg_joint: origin xyz=0.3 0.0 0.2 rpy=0.0 0.0 0.0 -> xyz=0.0 -0.3 0.2 rpy=0.0 0.0 0.0
- joint base_to_head_left_joint: origin xyz=0.5 0.17 1.7 rpy=0.0 0.0 0.0 -> xyz=0.17 -0.5 1.7 rpy=0.0 0.0 0.0
- joint base_to_head_right_joint: origin xyz=0.5 -0.17 1.7 rpy=0.0 0.0 0.0 -> xyz=-0.17 -0.5 1.7 rpy=0.0 0.0 0.0
- joint base_to_left_wheel_joint: axis 0.0 1.0 0.0 -> 0.0 0.0 1.0; origin xyz=-0.3 0.3 0.11 rpy=0 0 0 -> xyz=-0.3 0.3 0.11 rpy=1.57075 0 0.0
- joint base_to_lidar_joint: origin xyz=0.6 0.0 0.25 rpy=0.0 0.0 0.0 -> xyz=0.0 -0.6 0.25 rpy=0.0 0.0 0.0
- joint base_to_right_wheel_joint: axis 0.0 1.0 0.0 -> 0.0 0.0 1.0; origin xyz=-0.3 -0.3 0.11 rpy=0 0 0 -> xyz=-0.3 0.3 0.11 rpy=0.0 1.57075 0.0
