Commit message: mapping and localization added
mapping localization with slam_toolbox and edited all project

File: urdf/my_robot3.urdf (robot description, URDF)
Before this commit: robot myRobot, 12 links, 11 joints
Links:
- link lidar_link: geometry collision box size=0.2 0.2 0.15; visual box size=0.2 0.2 0.15

Commit message: entegreted amr_mini to my_robot project

File: urdf/my_robot3.urdf (robot description, URDF)
Before this commit: robot myRobot, 12 links, 11 joints
Joints:
- joint base_to_footprint_joint: origin xyz=0.0 0.0 0.0 rpy=0.0 0.0 0.0 -> xyz=0.0 0.0 0.01 rpy=0.0 0.0 0.0
